File: KiCAD/CC1200_Hat.kicad_pcb (KiCad board)
At the start: 4 copper layers, 65.1 x 30.2 mm, 86 parts, among them P1 OLED, P2 Nextion, P3 SMA, P4 STLink, P5 USB_C_Plug_USB2.0, U1 CC1200, U3 TLV70233_SOT23-5, U4 USBLC6-2, U6 STM32F411CEUx, X1 40MHz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

Commit message: cleanup/update
- schematic/pcb cleanup
- WIP PN assignment
- KiCAD version update
Parts:
- removed AE1: CERAMIC_ANTENNA, M17:ANT1204
- removed C28: 1n, Capacitor_SMD:C_0402_1005Metric
- removed JP1: OLED_P1, Jumper:SolderJumper-3_P1.3mm_Bridged2Bar12_RoundedPad1.0x1.5mm
- removed JP2: OLED_P2, Jumper:SolderJumper-3_P1.3mm_Bridged2Bar12_RoundedPad1.0x1.5mm
- removed P1: OLED, Connector_PinHeader_2.54mm:PinHeader_1x04_P2.54mm_Vertical
- removed P2: Nextion, Connector_PinHeader_2.54mm:PinHeader_1x04_P2.54mm_Vertical
- removed P4: STLink, Connector_PinHeader_2.54mm:PinHeader_1x05_P2.54mm_Vertical
- removed R10, R2: 1k, Resistor_SMD:R_0402_1005Metric
- removed REF**: OSHW-Logo2_14.6x12mm_SilkScreen, Symbol:OSHW-Logo2_14.6x12mm_SilkScreen
- removed Ref**: Val**, M17:M17-logo
- added J1: SWD, Connector_PinHeader_2.54mm:PinHeader_1x04_P2.54mm_Vertical, F.Cu at (201.9, 113.9)
- moved D2 15.6 mm to (192.0, 133.3)
- moved R11 13.3 mm to (192.0, 132.1), turned to 0 degrees
- moved D1 8.89 mm to (198.4, 133.3)
- moved R13 6.84 mm to (211.4, 132.1)
- moved R18 6.60 mm to (198.5, 132.1), turned to 180 degrees
- moved D4 4.48 mm to (211.4, 133.3), turned to 0 degrees
- moved L3 3.26 mm to (166.6, 123.8)
- moved D3 2.23 mm to (204.9, 133.3)
- moved C25 1.90 mm to (202.5, 129.9), turned to 0 degrees
- moved C4 1.65 mm to (167.8, 119.3)
- moved L2 0.84 mm to (169.1, 119.3), turned to -90 degrees
- moved R12 0.76 mm to (204.9, 132.1), turned to 0 degrees
- moved C27 0.08 mm to (166.6, 126.0)
- moved P3 0.08 mm to (166.6, 131.2)
Connections:
- net /CC_nCS renamed /~{CC_CS}
- net /CC_nRST renamed /~{CC_RST}
- net /xUDN renamed Net-(P5-D--PadA7)
- net /xUDP renamed Net-(P5-D+-PadA6)
- net BOOT0 renamed /BOOT0
- net COS_LED renamed /RX_LED
- net Net-(U6-PH0) renamed /X1
- net Net-(U6-PH1) renamed /X2
- net PTT_LED renamed /TX_LED
- net RXD renamed /MCU_RX
- net SERVICE renamed /SVC_LED
- net TXD renamed /MCU_TX
- net USB_DN renamed /USB_DN
- net USB_DP renamed /USB_DP
- net nRST renamed /~{MCU_RST}
- PI1 pad 3: /OLED_SDA -> unconnected-(PI1-SDA/GPIO2-Pad3)
- PI1 pad 5: /OLED_SCL -> unconnected-(PI1-SCL/GPIO3-Pad5)
- U1 pad 30: unconnected-(U1-XOSC_Q1-Pad30) -> GND
- U6 pad 12: Net-(P2-Pin_3) -> unconnected-(U6-PA2-Pad12)
- U6 pad 13: Net-(P2-Pin_2) -> unconnected-(U6-PA3-Pad13)
Routing:
- net +5V: track 112.7 -> 79.7 mm
- net /OLED_SDA: track 31.2 -> 0.00 mm
- net /OLED_SCL: track 29.1 -> 0.00 mm
- net Net-(P2-Pin_3): track 21.8 -> 0.00 mm, vias 2 -> 0
- net Net-(P2-Pin_2): track 18.6 -> 0.00 mm, vias 2 -> 0
- net Net-(AE1-Pad1): track 7.91 -> 0.00 mm
- net Net-(JP1-C): track 5.05 -> 0.00 mm
- net Net-(JP2-C): track 4.97 -> 0.00 mm
- net /SVC_LED: track 7.87 -> 12.4 mm, vias 2 -> 0
- net +3.3V: track 53.5 -> 49.4 mm, vias 21 -> 19
- net Net-(C27-Pad2): track 4.62 -> 1.32 mm
- net Net-(C4-Pad2): track 2.66 -> 5.28 mm
- net /RX_LED: track 11.1 -> 8.77 mm, vias 2 -> 0
- net GND: track 2.19 -> 3.78 mm, vias 69 -> 106
- net /~{MCU_RST}: track 28.0 -> 26.6 mm
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Other:
- board text added: "CC1200 Shield"
- board text added: "REV B"
- board text added: "SP5WWP & DB9MAT M17 Foundation 2025 CC BY-NC-SA 4.0"
- board text added: "SWD"
- board text removed: "3v3"
- board text removed: "5v0"
- board text removed: "CC1200_Hat"
- board text removed: "M17 Team, CERN-OHL-W r1.0 01/2024"
- board text removed: "Nextion"
- board text removed: "OLED"
- board text removed: "RXD"
- board text removed: "SCL"
- board text removed: "SDA"
- board text removed: "ST-Link"
- board text removed: "TXD"

Commit message: minor updates
- pcb update - "PROG" button
- readme update
- WIP PN update
Parts:
- added SW1: PROG, Button_Switch_SMD:SW_Tactile_SPST_NO_Straight_CK_PTS636Sx25SMTRLFS, F.Cu at (211.2, 128.2)
Routing:
- net /BOOT0: track 21.2 -> 26.8 mm
- net +3.3V: track 49.4 -> 51.0 mm, vias 19 -> 20
Other:
- board text added: "PROG"

Commit message: PN assignment
Parts:
- L10: value 10u -> 4u7
