File: KiCAD/CC1200_Hat.kicad_sch (KiCad schematic)
At the start: 84 parts, among them P1 OLED, P2 Nextion, P3 SMA, P4 STLink, P5 USB_C_Plug_USB2.0, U1 CC1200, U3 TLV70233_SOT23-5, U4 USBLC6-2, U6 STM32F411CEUx, X1 40MHz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

Commit message: cleanup/update
- schematic/pcb cleanup
- WIP PN assignment
- KiCAD version update
Parts:
- removed AE1: CERAMIC_ANTENNA, M17:ANT1204, symbol mmdvm_hs-hat-rescue:Antenna_Dipole-RESCUE-mmdvm_hs-hat
- removed C28: 1n, Capacitor_SMD:C_0402_1005Metric, symbol Device:C_Small
- removed JP1: OLED_P1, Jumper:SolderJumper-3_P1.3mm_Bridged2Bar12_RoundedPad1.0x1.5mm, symbol Jumper:Jumper_3_Bridged12
- removed JP2: OLED_P2, Jumper:SolderJumper-3_P1.3mm_Bridged2Bar12_RoundedPad1.0x1.5mm, symbol Jumper:Jumper_3_Bridged12
- removed P1: OLED, Connector_PinHeader_2.54mm:PinHeader_1x04_P2.54mm_Vertical, symbol Connector_Generic:Conn_01x04
- removed P2: Nextion, Connector_PinHeader_2.54mm:PinHeader_1x04_P2.54mm_Vertical, symbol Connector_Generic:Conn_01x04
- removed P4: STLink, Connector_PinHeader_2.54mm:PinHeader_1x05_P2.54mm_Vertical, symbol Connector_Generic:Conn_01x05
- removed R10, R2: 1k, Resistor_SMD:R_0402_1005Metric, symbol Device:R_Small
- added J1: SWD, Connector_PinHeader_2.54mm:PinHeader_1x04_P2.54mm_Vertical, symbol Connector_Generic:Conn_01x04
- C14, C35: MPN (none) -> VJ0402V104ZXJCW1BC; PN (none) -> 77-VJ0402V104ZXJCBC
- C21, C23: PN (none) -> 81-GJM1555C1H200FB1D; SPN 81-GJM1555C1H200FB1D -> (none); SPR Mouser -> (none)
- C24, C25: MFR Vishay / Vitramon -> (none); PN (none) -> 77-VJ0402V104ZXJCBC; SPN 77-VJ0402V104ZXJCBC -> (none); SPR Mouser -> (none)
- C26: PN (none) -> 77-VJ0402V104ZXJCBC; SPN 77-VJ0402V104ZXJCBC -> (none); SPR Mouser -> (none)
- C27: PN (none) -> 77-VJ0402V104ZXJCBC; SPN 77-VJ0402V104ZXJCBC -> (none); SPR Mouser -> (none); now fitted; now in the parts list
- D1: PN (none) -> 604-APHHS1005SURCK; SPN 604-APHHS1005SURCK -> (none); SPR Mouser -> (none)
- D2: PN (none) -> 604-APHHS1005CGCK; SPN 604-APHHS1005CGCK -> (none); SPR Mouser -> (none)
- D3: PN (none) -> 604-APG1005SYCT; SPN 604-APG1005SYCT -> (none); SPR Mouser -> (none)
- D4: MFR Kingbright -> (none); PN (none) -> 604-APHHS1005SURCK; SPN 604-APHHS1005SURCK -> (none); SPR Mouser -> (none)
- P3: now fitted; now in the parts list
- P5: MPN (none) -> TYPE-C-31-M-12; PN (none) -> C165948
- PI1: now left out of the parts list
- R11, R12, R13, R18: MFR Panasonic -> (none); PN (none) -> 667-ERJ-PA2D1001X; SPN 667-ERJ-PA2D1001X -> (none); SPR Mouser -> (none)
- R22, R23, R25, R26: PN (none) -> 71-CRCW0402-10K-E3; SPN 71-CRCW0402-10K-E3 -> (none); SPR Mouser -> (none)
- X1: PN (none) -> 815-FT2MNTUM-40.0-T1
- Y1: MPN (none) -> EB2532YA08-25T; PN (none) -> 669-EB2532YA08-25T
Connections:
- net GND: now also U1.30 (XOSC_Q1), J1.4 (Pin_4)
- net X1: now reaches C21.1, U6.5 (PH0), Y1.1
- net X2: now reaches C23.1, U6.6 (PH1), Y1.3
- net at U6.34 (PA13): now also J1.1 (Pin_1)
- net at U6.37 (PA14): now also J1.2 (Pin_2)
- net CC_nCS renamed ~{CC_CS}
- net CC_nRST renamed ~{CC_RST}
- net COS_LED renamed RX_LED
- net OLED_SCL: no longer names the net of PI1.5 (SCL/GPIO3)
- net OLED_SDA: no longer names the net of PI1.3 (SDA/GPIO2)
- net PTT_LED renamed TX_LED
- net RXD renamed MCU_RX
- net SERVICE renamed SVC_LED
- net TXD renamed MCU_TX
- net nRST renamed ~{MCU_RST}
- net ~{MCU_RST}: now also J1.3 (Pin_3)
- net xUDN: no longer names the net of P5.A7 (D-), P5.B7 (D-), U4.1 (IO1)
- net xUDP: no longer names the net of P5.A6 (D+), P5.B6 (D+), U4.3 (IO2)
- no-connect marks 29 -> 45
Other:
- note added: "BOOT1"
- note added: "USB is optional"
- note removed: "CC1200 Hotspot Pi Hat"
- note removed: "Install either"
- note removed: "USB is optional."
- company: DB9MAT, SP5WWP, M17 Team -> M17 Foundation
- title: CC1200_Hat -> CC1200 RPi Zero Shield
- moved on the sheet: C1, C10, C11, C12, C13, C14, C15, C16, C17, C18, C19, C2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

Commit message: minor updates
- pcb update - "PROG" button
- readme update
- WIP PN update
Parts:
- added SW1: PROG, Button_Switch_SMD:SW_Tactile_SPST_NO_Straight_CK_PTS636Sx25SMTRLFS, symbol Switch:SW_Push
- C27: MFR Vishay / Vitramon -> (none)
Connections:
- net +3.3V: now also SW1.2
- net BOOT0: now also SW1.1
Other:
- moved on the sheet: R9
Changed lines of the file:
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@@
 	(title_block
 		(title "CC1200 RPi Zero Shield")
-		(date "06-02-2025")
+		(date "7-02-2025")
 		(rev "B")
 		(company "M17 Foundation")
@@
 	)
 	(junction
+		(at 48.26 114.3)
+		(diameter 0)
+		(color 0 0 0 0)
+	)
+	(junction
 		(at 173.99 182.88)
 		(diameter 0)
@@
 	)
 	(junction
+		(at 38.1 109.22)
+		(diameter 0)
+		(color 0 0 0 0)
+	)
+	(junction
 		(at 212.09 132.08)
 		(diameter 0)
@@
 	(wire
 		(pts
-			(xy 40.64 114.3) (xy 38.1 114.3)
-		)
-		(stroke
-			(width 0)
-			(type default)
-		)
-	)
-	(wire
-		(pts
 			(xy 194.31 157.48) (xy 194.31 160.02)
 		)
@@
 	(wire
 		(pts
+			(xy 34.29 114.3) (xy 34.29 109.22)
+		)
+		(stroke
+			(width 0)
+			(type default)
+		)
+	)
+	(wire
+		(pts
 			(xy 91.44 19.05) (xy 91.44 21.59)
 		)
@@
 	(wire
 		(pts
+			(xy 34.29 109.22) (xy 38.1 109.22)
+		)
+		(stroke
+			(width 0)
+			(type default)
+		)
+	)
+	(wire
+		(pts
 			(xy 134.62 123.19) (xy 134.62 121.92)
 		)
@@
 	(wire
 		(pts
-			(xy 45.72 114.3) (xy 58.42 114.3)
+			(xy 45.72 114.3) (xy 48.26 114.3)
 		)
 		(stroke
@@
 	(wire
 		(pts
+			(xy 48.26 114.3) (xy 48.26 116.84)
+		)
+		(stroke
+			(width 0)
+			(type default)
+		)
+	)
+	(wire
+		(pts
 			(xy 161.29 54.61) (xy 161.29 52.07)
 		)
@@
 	(wire
 		(pts
+			(xy 35.56 114.3) (xy 34.29 114.3)
+		)
+		(stroke
+			(width 0)
+			(type default)
+		)
+	)
+	(wire
+		(pts
 			(xy 180.34 72.39) (xy 184.15 72.39)
 		)
@@
 	(wire
 		(pts
+			(xy 48.26 123.19) (xy 48.26 121.92)
+		)
+		(stroke
+			(width 0)
+			(type default)
+		)
+	)
+	(wire
+		(pts
 			(xy 24.13 54.61) (xy 21.59 54.61)
 		)
@@
 	(wire
 		(pts
+			(xy 48.26 114.3) (xy 58.42 114.3)
+		)
+		(stroke
+			(width 0)
+			(type default)
+		)
+	)
+	(wire
+		(pts
 			(xy 78.74 101.6) (xy 81.28 101.6)
 		)
@@
 	(wire
 		(pts
-			(xy 38.1 114.3) (xy 38.1 116.84)
-		)
-		(stroke
-			(width 0)
-			(type default)
-		)
-	)
-	(wire
-		(pts
 			(xy 172.72 72.39) (xy 172.72 82.55)
 		)
@@
 	(text "BOOT1"
 		(exclude_from_sim no)
-		(at 39.37 140.97 0)
+		(at 52.07 140.97 0)
 		(effects
 			(font
@@
 		(lib_id "Device:C_Small")
 		(at 186.69 72.39 270)
-		(mirror x)
 		(unit 1)
 		(exclude_from_sim no)
@@
 		(dnp no)
 		(property "Reference" "C27"
-			(at 189.23 71.755 0)
+			(at 186.69 67.31 90)
 			(effects
 				(font
 					(size 1.27 1.27)
 				)
-				(justify left)
 			)
 		)
 		(property "Value" "1n"
-			(at 184.15 71.755 0)
+			(at 185.42 69.85 90)
 			(effects
 				(font
@@
 			)
 		)
-		(property "MFR" "Vishay / Vitramon"
-			(at 124.46 207.01 0)
-			(effects
-				(font
-					(size 1.27 1.27)
-				)
-				(hide yes)
-			)
-		)
 		(property "MPN" "VJ0402V104ZXJCW1BC"
-			(at 124.46 207.01 0)
+			(at 124.46 -62.23 0)
 			(effects
 				(font
@@
 	)
 	(symbol
+		(lib_id "Switch:SW_Push")
+		(at 40.64 114.3 180)
+		(unit 1)
+		(exclude_from_sim no)
+		(in_bom yes)
+		(on_board yes)
+		(dnp no)
+		(property "Reference" "SW1"
+			(at 40.64 111.76 0)
+			(effects
+				(font
+					(size 1.27 1.27)
+				)
+			)
+		)
+		(property "Value" "PROG"
+			(at 40.64 119.38 0)
+			(effects
+				(font
+					(size 1.27 1.27)
+				)
+			)
+		)
+		(property "Footprint" "Button_Switch_SMD:SW_Tactile_SPST_NO_Straight_CK_PTS636Sx25SMTRLFS"
+			(at 40.64 119.38 0)
+			(effects
+				(font
+					(size 1.27 1.27)
+				)
+				(hide yes)
+			)
+		)
+		(property "Datasheet" "~"
+			(at 40.64 119.38 0)
+			(effects
+				(font
+					(size 1.27 1.27)
+				)
+				(hide yes)
+			)
+		)
+		(property "Description" "Push button switch, generic, two pins"
+			(at 40.64 114.3 0)
+			(effects
+				(font
+					(size 1.27 1.27)
+				)
+				(hide yes)
+			)
+		)
+		(property "PN" "611-PTS636SM43JSMTRL"
+			(at 40.64 114.3 0)
+			(effects
+				(font
+					(size 1.524 1.524)
+				)
+				(hide yes)
+			)
+		)
+		(property "MPN" "PTS636SM43JSMTR LFS"
+			(at 40.64 114.3 0)
+			(effects
+				(font
+					(size 1.524 1.524)
+				)
+				(hide yes)
+			)
+		)
+		(pin "2"
+		)
+		(pin "1"
+		)
+		(instances
+			(project ""
+				(path "/64f5051f-1b71-4f29-a149-913e6a95d2cf"
+					(reference "SW1")
+					(unit 1)
+				)
+			)
+		)
+	)
+	(symbol
 		(lib_id "power:GND")
 		(at 55.88 190.5 0)
@@
 	)
 	(symbol
-		(lib_id "power:GND")
-		(at 38.1 116.84 0)
-		(mirror y)
-		(unit 1)
-		(exclude_from_sim no)
-		(in_bom yes)
-		(on_board yes)
-		(dnp no)
-		(property "Reference" "#PWR049"
-			(at 38.1 123.19 0)
-			(effects
-				(font
-					(size 1.27 1.27)
-				)
-				(hide yes)
-			)
-		)
-		(property "Value" "GND"
-			(at 38.1 120.65 0)
-			(effects
-				(font
-					(size 1.27 1.27)
-				)
-			)
-		)
-		(property "Footprint" ""
-			(at 38.1 116.84 0)
-			(effects
-				(font
-					(size 1.27 1.27)
-				)
-			)
-		)
-		(property "Datasheet" ""
-			(at 38.1 116.84 0)
-			(effects
-				(font
-					(size 1.27 1.27)
-				)
-			)
-		)
-		(property "Description" ""
-			(at 38.1 116.84 0)
-			(effects
-				(font
-					(size 1.27 1.27)
-				)
-				(hide yes)
-			)
-		)
-		(pin "1"
-		)
-		(instances
-			(project "CC1200_Hat"
-				(path "/64f5051f-1b71-4f29-a149-913e6a95d2cf"
-					(reference "#PWR049")
-					(unit 1)
-				)
-			)
-		)
-	)
-	(symbol
 		(lib_id "Device:C_Small")
 		(at 130.81 184.15 0)
@@
 	(symbol
 		(lib_id "Device:R_Small")
-		(at 43.18 114.3 90)
+		(at 48.26 119.38 180)
 		(unit 1)
 		(exclude_from_sim no)
@@
 		(dnp no)
 		(property "Reference" "R9"
-			(at 43.18 111.76 90)
+			(at 45.72 119.38 90)
 			(effects
 				(font
@@
 		)
 		(property "Value" "10k"
-			(at 43.18 114.3 90)
+			(at 48.26 119.38 90)
 			(effects
 				(font
@@
 		)
 		(property "Footprint" "Resistor_SMD:R_0402_1005Metric"
-			(at 43.18 114.3 0)
+			(at 48.26 119.38 0)
 			(effects
 				(font
@@
 		)
 		(property "Datasheet" "~"
-			(at 43.18 114.3 0)
+			(at 48.26 119.38 0)
 			(effects
 				(font
@@
 		)
 		(property "Description" ""
-			(at 43.18 114.3 0)
+			(at 48.26 119.38 0)
 			(effects
 				(font
@@
 					(unit 1)
 				)
+			)
+		)
+	)
+	(symbol
+		(lib_id "power:GND")
+		(at 48.26 123.19 0)
+		(mirror y)
+		(unit 1)
+		(exclude_from_sim no)
+		(in_bom yes)
+		(on_board yes)
+		(dnp no)
+		(property "Reference" "#PWR036"
+			(at 48.26 129.54 0)
+			(effects
+				(font
+					(size 1.27 1.27)
+				)
+				(hide yes)
+			)
+		)
+		(property "Value" "GND"
+			(at 48.26 127 0)
+			(effects
+				(font
+					(size 1.27 1.27)
+				)
+			)
+		)
+		(property "Footprint" ""
+			(at 48.26 123.19 0)
+			(effects
+				(font
+					(size 1.27 1.27)
+				)
+			)
+		)
+		(property "Datasheet" ""
+			(at 48.26 123.19 0)
+			(effects
+				(font
+					(size 1.27 1.27)
+				)
+			)
+		)
+		(property "Description" ""
+			(at 48.26 123.19 0)
+			(effects
+				(font
+					(size 1.27 1.27)
+				)
+				(hide yes)
+			)
+		)
+		(pin "1"
+		)
+		(instances
+			(project "CC1200_Hat"
+				(path "/64f5051f-1b71-4f29-a149-913e6a95d2cf"
+					(reference "#PWR036")
+					(unit 1)
+				)

Commit message: PN assignment
Parts:
- C1: MPN (none) -> GCM1555C1H2R2BA6J; PN (none) -> 81-GCM1555C1H2R2BA6J
- C10, C11, C15, C17, C18, C19, C20, C22, C30, C32, C33, C34: MPN (none) -> GCM155L8EH473KE7D; PN (none) -> 81-GCM155L8EH473KE7D
- C12, C6: MPN (none) -> 0402B103K6R3CT; PN (none) -> 791-0402B103K6R3CT
- C13: MPN (none) -> CGA2B3X5R1A224MB; PN (none) -> 810-CGA2B3X5R1A224MB
- C14, C27: MPN VJ0402V104ZXJCW1BC -> GRT1555C1E102JA2J; PN 77-VJ0402V104ZXJCBC -> 77-81-GRT1555C1E102JA2J
- C16: MPN (none) -> 885012205026; PN (none) -> 710-885012205026
- C2: MPN (none) -> GRM1555C2A390JA1D; PN (none) -> 81-GRM1555C2A390JA1D
- C29: MPN (none) -> CL10A106KQ8NNNC; PN (none) -> 187-CL10A106KQ8NNNC
- C3, C8, C9: MPN (none) -> GJM1555C1H5R1DB1D; PN (none) -> 81-GJM1555C1H5R1DB1D
- C31: MPN (none) -> CL10A225KO8NNWC; PN (none) -> 187-CL10A225KO8NNWC
- C4: MPN (none) -> GCM1555C1H6R2BA6D; PN (none) -> 81-GCM1555C1H6R2BA6D
- C5: MPN (none) -> 04025A560JAT4A; PN (none) -> 581-04025A560JAT4A
- C7: MPN (none) -> CL05C101JB5NNNC; PN (none) -> 187-CL05C101JB5NNNC
- D5, D6: MPN (none) -> BAT60AE6327XT; PN (none) -> 726-BAT60AE6327XT
- J1, PI1: MPN (none) -> -; PN (none) -> -
- L1, L9: MPN (none) -> LQG15HZ15NJ02D; PN (none) -> 81-LQG15HZ15NJ02D
- L10: value 10u -> 4u7; MPN (none) -> PLEA67BCA4R7M-1PT00; PN (none) -> 810-PLEA67BCA4R7M1PT
- L2: MPN (none) -> LQG15WZ43NJ02D; PN (none) -> 81-LQG15WZ43NJ02D
- L3: MPN (none) -> LQG15HZ22NH02D; PN (none) -> 81-LQG15HZ22NH02D
- L4, L7: MPN (none) -> LCCI0402J56NGTAR; PN (none) -> 581-LCCI0402J56NGTAR
- L6, L8: MPN (none) -> LQG15HN27NJ02D; PN (none) -> 81-LQG15HN27NJ02D
- P3: MPN (none) -> RF2-04A-T-00-50-G; PN (none) -> 737-RF204AT0050G
- R1, R7, R9: MPN (none) -> RC0402JR-1010KL; PN (none) -> 603-RC0402JR-1010KL
- R14: MPN (none) -> RK73B1ETTP563J; PN (none) -> 660-RK73B1ETTP563J
- R24: MPN (none) -> AC0402JR-7W1K5L; PN (none) -> 603-AC0402JR-7W1K5L
- R3: MPN (none) -> ERJ-2GEJ180X; PN (none) -> 667-ERJ-2GEJ180X
- R4, R5, R6: MPN (none) -> CR0402AJW-101GLF; PN (none) -> 652-CR0402AJW-101GLF
- U1: MPN (none) -> CC1200RHBR; PN (none) -> 595-CC1200RHBR
- U3: MPN (none) -> TLV70233PDBVR; PN (none) -> 595-TLV70233PDBVR
- U4: MPN (none) -> USBLC6-2SC6; PN (none) -> 511-USBLC6-2SC6
- U6: MPN (none) -> STM32F411CEU6; PN (none) -> 511-STM32F411CEU6
- Y1: PN 669-EB2532YA08-25T -> 669-EB2532YA08-25T

Commit message: MPN fixes for Mouser
Parts:
- C1: MPN GCM1555C1H2R2BA6J -> GCM1555C1H2R2BA16J
- C13: MPN CGA2B3X5R1A224MB -> CGA2B3X5R1A224M050BB
- C21, C23: MPN GJM1555C1H200FB01D -> C0402C120J5GACTU; PN 81-GJM1555C1H200FB1D -> 80-C0402C120J5G
- D1: MPN APHHS1005SURCK -> APHHS1005QBC/D; PN 604-APHHS1005SURCK -> 604-APHHS1005QBCD
- R22, R23: MPN CRCW040210K0FKED -> RC0402FR-075K1L; PN 71-CRCW0402-10K-E3 -> 603-RC0402FR-075K1L
- Y1: MPN EB2532YA08-25T -> EB2532YA08-25.000M TR; PN 669-EB2532YA08-25T -> 669-EB2532YA08-25T
Changed lines of the file:
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@@
 	(title_block
 		(title "CC1200 RPi Zero Shield")
-		(date "7-02-2025")
+		(date "10-02-2025")
 		(rev "B")
 		(company "M17 Foundation")
@@
 			)
 		)
-		(property "MPN" "GJM1555C1H200FB01D"
+		(property "MPN" "C0402C120J5GACTU"
 			(at 292.1 195.58 0)
 			(effects
@@
 			)
 		)
-		(property "PN" "81-GJM1555C1H200FB1D"
+		(property "PN" "80-C0402C120J5G"
 			(at 292.1 195.58 0)
 			(effects
@@
 			)
 		)
-		(property "MPN" "GJM1555C1H200FB01D"
+		(property "MPN" "C0402C120J5GACTU"
 			(at -35.56 195.58 0)
 			(effects
@@
 			)
 		)
-		(property "PN" "81-GJM1555C1H200FB1D"
+		(property "PN" "80-C0402C120J5G"
 			(at -35.56 195.58 0)
 			(effects
@@
 			)
 		)
-		(property "MPN" "APHHS1005SURCK"
+		(property "MPN" "APHHS1005QBC/D"
 			(at 434.34 340.36 0)
 			(effects
@@
 			)
 		)
-		(property "PN" "604-APHHS1005SURCK"
+		(property "PN" "604-APHHS1005QBCD"
 			(at 168.91 190.5 0)
 			(effects
@@
 			)
 		)
-		(property "MPN" "CRCW040210K0FKED"
+		(property "MPN" "RC0402FR-075K1L"
 			(at 313.69 176.53 0)
 			(effects
@@
 			)
 		)
-		(property "PN" "71-CRCW0402-10K-E3"
+		(property "PN" "603-RC0402FR-075K1L"
 			(at 215.9 121.92 0)
 			(effects
@@
 			)
 		)
-		(property "MPN" "CRCW040210K0FKED"
+		(property "MPN" "RC0402FR-075K1L"
 			(at 313.69 179.07 0)
 			(effects
@@
 			)
 		)
-		(property "PN" "71-CRCW0402-10K-E3"
+		(property "PN" "603-RC0402FR-075K1L"
 			(at 215.9 124.46 0)
 			(effects
@@
 			)
 		)
-		(property "MPN" "CGA2B3X5R1A224MB"
+		(property "MPN" "CGA2B3X5R1A224M050BB"
 			(at 133.35 62.23 0)
 			(effects
@@
 			)
 		)
-		(property "PN" "669-EB2532YA08-25T "
+		(property "PN" "669-EB2532YA08-25T"
 			(at 134.62 125.73 0)
 			(effects
@@
 			)
 		)
-		(property "MPN" "EB2532YA08-25T "
+		(property "MPN" "EB2532YA08-25.000M TR"
 			(at 134.62 125.73 0)
 			(effects
@@
 			)
 		)
-		(property "MPN" "GCM1555C1H2R2BA6J"
+		(property "MPN" "GCM1555C1H2R2BA16J"
 			(at 157.48 80.01 0)
 			(effects

Commit message: updates
- KiCAD version bump to 9.0
- BOM value update for R25 & R26
Parts:
- R25, R26: MPN CRCW040210K0FKED -> CR0402-FX-27R0GLF; PN 71-CRCW0402-10K-E3 -> 652-CR0402FX-27R0GLF
Changed lines of the file:
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@@
 (kicad_sch
-	(version 20231120)
+	(version 20250114)
 	(generator "eeschema")
-	(generator_version "8.0")
+	(generator_version "9.0")
 	(paper "A4")
 	(title_block
@@
 		(comment 1 "Wojciech SP5WWP, Mathis DB9MAT")
 	)
+	(text "BOOT1"
+		(exclude_from_sim no)
+		(at 52.07 140.97 0)
+		(effects
+			(font
+				(size 1.524 1.524)
+			)
+		)
+	)
+	(text "USB is optional"
+		(exclude_from_sim no)
+		(at 248.92 162.56 0)
+		(effects
+			(font
+				(size 2.4892 2.4892)
+				(thickness 0.3112)
+			)
+			(justify left bottom)
+		)
+	)
 	(junction
 		(at 170.18 52.07)
@@
 		)
 	)
-	(text "BOOT1"
-		(exclude_from_sim no)
-		(at 52.07 140.97 0)
-		(effects
-			(font
-				(size 1.524 1.524)
-			)
-		)
-	)
-	(text "USB is optional"
-		(exclude_from_sim no)
-		(at 248.92 162.56 0)
-		(effects
-			(font
-				(size 2.4892 2.4892)
-				(thickness 0.3112)
-			)
-			(justify left bottom)
-		)
-	)
 	(label "USB_DP"
 		(at 271.78 137.16 0)
@@
 			)
 		)
-		(property "MPN" "CRCW040210K0FKED"
+		(property "MPN" "CR0402-FX-27R0GLF"
 			(at 359.41 186.69 0)
 			(effects
@@
 			)
 		)
-		(property "PN" "71-CRCW0402-10K-E3"
+		(property "PN" "652-CR0402FX-27R0GLF"
 			(at 261.62 132.08 0)
 			(effects
@@
 			)
 		)
-		(property "MPN" "CRCW040210K0FKED"
+		(property "MPN" "CR0402-FX-27R0GLF"
 			(at 359.41 191.77 0)
 			(effects
@@
 			)
 		)
-		(property "PN" "71-CRCW0402-10K-E3"
+		(property "PN" "652-CR0402FX-27R0GLF"
 			(at 261.62 137.16 0)
 			(effects
@@
 		)
 	)
+	(embedded_fonts no)
 )
